File: Workspace/Jenny Meier/Schema/UART/_saved_UART.sch (KiCad schematic (older format))
At the start: 13 parts

Commit message: Uart
Parts:
- added R?: 10k, symbol Device:R
Connections:
- net +5V: now also R?.2
- net at U?.2 (EEDATA): now also R?.1
- no-connect marks 0 -> 9
Changed lines of the file:
@@
 P 5450 3450
 F 0 "#PWR?" H 5450 3300 50  0001 C CNN
-F 1 "+3.3V" V 5465 3578 50  0000 L CNN
+F 1 "+3.3V" H 5465 3623 50  0000 C CNN
 F 2 "" H 5450 3450 50  0001 C CNN
 F 3 "" H 5450 3450 50  0001 C CNN
 	1    5450 3450
-	0    1    1    0
+	1    0    0    -1
 $EndComp
 $Comp
@@
 P 5450 4950
 F 0 "#PWR?" H 5450 4800 50  0001 C CNN
-F 1 "+3.3V" V 5465 5078 50  0000 L CNN
+F 1 "+3.3V" H 5465 5123 50  0000 C CNN
 F 2 "" H 5450 4950 50  0001 C CNN
 F 3 "" H 5450 4950 50  0001 C CNN
 	1    5450 4950
-	0    1    1    0
+	1    0    0    -1
 $EndComp
 Wire Wire Line
@@
 Wire Wire Line
 	5550 2250 5300 2250
+NoConn ~ 3500 4550
+NoConn ~ 3500 4650
+NoConn ~ 5300 2350
+NoConn ~ 5300 2450
+NoConn ~ 5300 2550
+NoConn ~ 5300 2650
+NoConn ~ 5300 2750
+NoConn ~ 5300 2850
+$Comp
+L Device:R R?
+U 1 1 5E74B89F
+P 3200 4750
+F 0 "R?" V 3100 4550 50  0000 L CNN
+F 1 "10k" V 3100 4750 50  0000 L CNN
+F 2 "" V 3130 4750 50  0001 C CNN
+F 3 "~" H 3200 4750 50  0001 C CNN
+	1    3200 4750
+	0    1    1    0
+$EndComp
+$Comp
+L power:+5V #PWR?
+U 1 1 5E74B93F
+P 2900 4700
+F 0 "#PWR?" H 2900 4550 50  0001 C CNN
+F 1 "+5V" H 2915 4873 50  0000 C CNN
+F 2 "" H 2900 4700 50  0001 C CNN
+F 3 "" H 2900 4700 50  0001 C CNN
+	1    2900 4700
+	1    0    0    -1
+$EndComp
+Wire Wire Line
+	3350 4750 3500 4750
+Wire Wire Line
+	3050 4750 2900 4750
+Wire Wire Line
+	2900 4750 2900 4700
+NoConn ~ 3500 4250
 $EndSCHEMATC
